Commit message: arm_controller working with moveIt!

File: phantomx_reactor_arm_description/urdf/phantomx_reactor_wrist.urdf.xacro (robot description, xacro)
@@ -109,4 +109,12 @@
 			</collision>
 		</link>
+		<joint name="${prefix}shoulder_pitch_mimic_joint" type="revolute">
+			<origin xyz="0 0 0.0265" rpy="${PI/2} 0 0" />
+			<parent link="${prefix}shoulder_link" />
+			<child link="dummy_shoulder_link" />
+			<axis xyz="0 0 -1" />
+			<limit effort="3.0" velocity="6.178465545" lower="${shoulder_pitch_joint_lower_limit}" upper="${shoulder_pitch_joint_upper_limit}" />
+		</joint>
+		<link name="dummy_shoulder_link" />
 	    <!-- ELBOW PITCH-->
 		<joint name="${prefix}elbow_pitch_joint" type="revolute">
@@ -140,4 +148,11 @@
 			</collision>
 		</link>
+		<joint name="${prefix}elbow_pitch_mimic_joint" type="revolute">
+			<origin xyz="0.0385 0.1445 0" rpy="-${PI/2} 0 0" />
+			<parent link="${prefix}bicep_link" />
+			<child link="dummy_elbow_link" />
+			<axis xyz="0 1 0" /> <limit effort="3.0" velocity="6.178465545" lower="${elbow_pitch_joint_lower_limit}" upper="${elbow_pitch_joint_upper_limit}" />
+		</joint>
+		<link name="dummy_elbow_link" />
 		<!-- WRIST PITCH-->
 		<joint name="${prefix}wrist_pitch_joint" type="revolute">
